Commit message: Transformation du topic /ur5/vacuum_gripper/grasp en un service grasp

File: ur_icam_description/urdf/ur5.urdf.xacro (robot description, xacro)
@@ -1,74 +1,82 @@
 <?xml version="1.0"?>
 <robot xmlns:xacro="http://ros.org/wiki/xacro">
-  <xacro:include filename="$(find ur_description)/urdf/ur.transmission.xacro" />
-  <xacro:include filename="$(find ur_description)/urdf/ur.gazebo.xacro" />
+  <xacro:include filename="$(find ur_description)/urdf/ur.transmission.xacro"/>
+  <xacro:include filename="$(find ur_description)/urdf/ur.gazebo.xacro"/>
   <!-- Inertia parameters -->
-  <xacro:property name="base_mass" value="4.0" />  <!-- This mass might be incorrect -->
-  <xacro:property name="shoulder_mass" value="3.7000" />
-  <xacro:property name="upper_arm_mass" value="8.3930" />
-  <xacro:property name="forearm_mass" value="2.2750" />
-  <xacro:property name="wrist_1_mass" value="1.2190" />
-  <xacro:property name="wrist_2_mass" value="1.2190" />
-  <xacro:property name="wrist_3_mass" value="0.1879" />
-  <xacro:property name="height3" value="1" /> <!-- Link 3 -->
-  <xacro:property name="camera_link" value="0.02" /> <!-- Size of square 'camera' box -->
-  <xacro:property name="axel_offset" value="0.05" /> <!-- Space btw top of beam and the each joint -->
-  <xacro:property name="shoulder_cog" value="0.0 0.00193 -0.02561" />
-  <xacro:property name="upper_arm_cog" value="0.0 -0.024201 0.2125" />
-  <xacro:property name="forearm_cog" value="0.0 0.0265 0.11993" />
-  <xacro:property name="wrist_1_cog" value="0.0 0.110949 0.01634" />
-  <xacro:property name="wrist_2_cog" value="0.0 0.0018 0.11099" />
-  <xacro:property name="wrist_3_cog" value="0.0 0.001159 0.0" />
+  <xacro:property name="base_mass" value="4.0"/>
+  <!-- This mass might be incorrect -->
+  <xacro:property name="shoulder_mass" value="3.7000"/>
+  <xacro:property name="upper_arm_mass" value="8.3930"/>
+  <xacro:property name="forearm_mass" value="2.2750"/>
+  <xacro:property name="wrist_1_mass" value="1.2190"/>
+  <xacro:property name="wrist_2_mass" value="1.2190"/>
+  <xacro:property name="wrist_3_mass" value="0.1879"/>
+  <xacro:property name="height3" value="1"/>
+  <!-- Link 3 -->
+  <xacro:property name="camera_link" value="0.02"/>
+  <!-- Size of square 'camera' box -->
+  <xacro:property name="axel_offset" value="0.05"/>
+  <!-- Space btw top of beam and the each joint -->
+  <xacro:property name="shoulder_cog" value="0.0 0.00193 -0.02561"/>
+  <xacro:property name="upper_arm_cog" value="0.0 -0.024201 0.2125"/>
+  <xacro:property name="forearm_cog" value="0.0 0.0265 0.11993"/>
+  <xacro:property name="wrist_1_cog" value="0.0 0.110949 0.01634"/>
+  <xacro:property name="wrist_2_cog" value="0.0 0.0018 0.11099"/>
+  <xacro:property name="wrist_3_cog" value="0.0 0.001159 0.0"/>
   <!-- Kinematic model -->
   <!-- Properties from urcontrol.conf -->
-  <!--
-    DH for UR5:
-    a = [0.00000, -0.42500, -0.39225,  0.00000,  0.00000,  0.0000]
-    d = [0.089159,  0.00000,  0.00000,  0.10915,  0.09465,  0.0823]
-    alpha = [ 1.570796327, 0, 0, 1.570796327, -1.570796327, 0 ]
-    q_home_offset = [0, -1.570796327, 0, -1.570796327, 0, 0]
-    joint_direction = [-1, -1, 1, 1, 1, 1]
-    mass = [3.7000, 8.3930, 2.2750, 1.2190, 1.2190, 0.1879]
-    center_of_mass = [ [0, -0.02561, 0.00193], [0.2125, 0, 0.11336], [0.11993, 0.0, 0.0265], [0, -0.0018, 0.01634], [0, 0.0018,0.01634], [0, 0, -0.001159] ]
+  <!-- DH for UR5: a = [0.00000, -0.42500, -0.39225, 0.00000, 0.00000, 0.0000] d = [0.089159, 0.00000, 0.00000, 0.10915, 0.09465, 0.0823] alpha = [ 1.570796327, 0, 0, 1.570796327, -1.570796327, 0 ] q_home_offset = [0, -1.570796327, 0, -1.570796327, 0,
+  0] joint_direction = [-1, -1, 1, 1, 1, 1] mass = [3.7000, 8.3930, 2.2750, 1.2190, 1.2190, 0.1879] center_of_mass = [ [0, -0.02561, 0.00193], [0.2125, 0, 0.11336], [0.11993, 0.0, 0.0265], [0, -0.0018, 0.01634], [0, 0.0018,0.01634], [0, 0, -0.001159] ]
   -->
-  <xacro:property name="ur5_d1" value="0.089159" />
-  <xacro:property name="ur5_a2" value="-0.42500" />
-  <xacro:property name="ur5_a3" value="-0.39225" />
-  <xacro:property name="ur5_d4" value="0.10915" />
-  <xacro:property name="ur5_d5" value="0.09465" />
-  <xacro:property name="ur5_d6" value="0.0823" />
+  <xacro:property name="ur5_d1" value="0.089159"/>
+  <xacro:property name="ur5_a2" value="-0.42500"/>
+  <xacro:property name="ur5_a3" value="-0.39225"/>
+  <xacro:property name="ur5_d4" value="0.10915"/>
+  <xacro:property name="ur5_d5" value="0.09465"/>
+  <xacro:property name="ur5_d6" value="0.0823"/>
   <!-- Arbitrary offsets for shoulder/elbow joints -->
-  <xacro:property name="shoulder_offset" value="0.13585" />  <!-- measured from model -->
-  <xacro:property name="elbow_offset" value="-0.1197" /> <!-- measured from model -->
+  <xacro:property name="shoulder_offset" value="0.13585"/>
+  <!-- measured from model -->
+  <xacro:property name="elbow_offset" value="-0.1197"/>
+  <!-- measured from model -->
   <!-- link lengths used in model -->
-  <xacro:property name="shoulder_height" value="${ur5_d1}" />
-  <xacro:property name="upper_arm_length" value="${-ur5_a2}" />
-  <xacro:property name="forearm_length" value="${-ur5_a3}" />
-  <xacro:property name="wrist_1_length" value="${ur5_d4 - elbow_offset - shoulder_offset}" />
-  <xacro:property name="wrist_2_length" value="${ur5_d5}" />
-  <xacro:property name="wrist_3_length" value="${ur5_d6}" />
+  <xacro:property name="shoulder_height" value="${ur5_d1}"/>
+  <xacro:property name="upper_arm_length" value="${-ur5_a2}"/>
+  <xacro:property name="forearm_length" value="${-ur5_a3}"/>
+  <xacro:property name="wrist_1_length" value="${ur5_d4 - elbow_offset - shoulder_offset}"/>
+  <xacro:property name="wrist_2_length" value="${ur5_d5}"/>
+  <xacro:property name="wrist_3_length" value="${ur5_d6}"/>
   <!--property name="shoulder_height" value="0.089159" /-->
-  <!--property name="shoulder_offset" value="0.13585" /-->  <!-- shoulder_offset - elbow_offset + wrist_1_length = 0.10915 -->
+  <!--property name="shoulder_offset" value="0.13585" /-->
+  <!-- shoulder_offset - elbow_offset + wrist_1_length = 0.10915 -->
   <!--property name="upper_arm_length" value="0.42500" /-->
-  <!--property name="elbow_offset" value="0.1197" /-->       <!-- CAD measured -->
+  <!--property name="elbow_offset" value="0.1197" /-->
+  <!-- CAD measured -->
   <!--property name="forearm_length" value="0.39225" /-->
-  <!--property name="wrist_1_length" value="0.093" /-->     <!-- CAD measured -->
-  <!--property name="wrist_2_length" value="0.09465" /-->   <!-- In CAD this distance is 0.930, but in the spec it is 0.09465 -->
+  <!--property name="wrist_1_length" value="0.093" /-->
+  <!-- CAD measured -->
+  <!--property name="wrist_2_length" value="0.09465" /-->
+  <!-- In CAD this distance is 0.930, but in the spec it is 0.09465 -->
   <!--property name="wrist_3_length" value="0.0823" /-->
-  <xacro:property name="shoulder_radius" value="0.060" />   <!-- manually measured -->
-  <xacro:property name="upper_arm_radius" value="0.054" />  <!-- manually measured -->
-  <xacro:property name="elbow_radius" value="0.060" />      <!-- manually measured -->
-  <xacro:property name="forearm_radius" value="0.040" />    <!-- manually measured -->
-  <xacro:property name="wrist_radius" value="0.045" />      <!-- manually measured -->
+  <xacro:property name="shoulder_radius" value="0.060"/>
+  <!-- manually measured -->
+  <xacro:property name="upper_arm_radius" value="0.054"/>
+  <!-- manually measured -->
+  <xacro:property name="elbow_radius" value="0.060"/>
+  <!-- manually measured -->
+  <xacro:property name="forearm_radius" value="0.040"/>
+  <!-- manually measured -->
+  <xacro:property name="wrist_radius" value="0.045"/>
+  <!-- manually measured -->
   <xacro:macro name="cylinder_inertial" params="radius length mass *origin">
     <inertial>
-      <mass value="${mass}" />
-      <xacro:insert_block name="origin" />
-      <inertia ixx="${0.0833333 * mass * (3 * radius * radius + length * length)}" ixy="0.0" ixz="0.0"
-        iyy="${0.0833333 * mass * (3 * radius * radius + length * length)}" iyz="0.0"
-        izz="${0.5 * mass * radius * radius}" />
+      <mass value="${mass}"/>
+      <xacro:insert_block name="origin"/>
+      <inertia ixx="${0.0833333 * mass * (3 * radius * radius + length * length)}" ixy="0.0" ixz="0.0" iyy="${0.0833333 * mass * (3 * radius * radius + length * length)}" iyz="0.0" izz="${0.5 * mass * radius * radius}"/>
     </inertial>
   </xacro:macro>
-  <xacro:macro name="ur5_robot" params="prefix joint_limited
+  <xacro:macro
+    name="ur5_robot"
+    params="prefix joint_limited
      shoulder_pan_lower_limit:=${-2*pi}    shoulder_pan_upper_limit:=${2*pi}
      shoulder_lift_lower_limit:=${-pi}    shoulder_lift_upper_limit:=${pi}
@@ -78,27 +86,27 @@
      wrist_3_lower_limit:=${-pi}    wrist_3_upper_limit:=${pi}
      transmission_hw_interface:=hardware_interface/PositionJointInterface">
-    <link name="${prefix}base_link" >
-      <visual>
-        <geometry>
-          <mesh filename="package://ur_description/meshes/ur5/visual/base.dae" />
-        </geometry>
-        <material name="LightGrey">
-          <color rgba="0.7 0.7 0.7 1.0"/>
-        </material>
-      </visual>
-      <collision>
-        <geometry>
-          <mesh filename="package://ur_description/meshes/ur5/collision/base.stl" />
+    <link name="${prefix}base_link">
+      <visual>
+        <geometry>
+          <mesh filename="package://ur_description/meshes/ur5/visual/base.dae"/>
+        </geometry>
+        <material name="LightGrey">
+          <color rgba="0.7 0.7 0.7 1.0"/>
+        </material>
+      </visual>
+      <collision>
+        <geometry>
+          <mesh filename="package://ur_description/meshes/ur5/collision/base.stl"/>
         </geometry>
       </collision>
       <xacro:cylinder_inertial radius="0.06" length="0.05" mass="${base_mass}">
-        <origin xyz="0.0 0.0 0.0" rpy="0 0 0" />
+        <origin xyz="0.0 0.0 0.0" rpy="0 0 0"/>
       </xacro:cylinder_inertial>
     </link>
     <joint name="${prefix}shoulder_pan_joint" type="revolute">
-      <parent link="${prefix}base_link" />
-      <child link = "${prefix}shoulder_link" />
-      <origin xyz="0.0 0.0 ${shoulder_height}" rpy="0.0 0.0 0.0" />
-      <axis xyz="0 0 1" />
+      <parent link="${prefix}base_link"/>
+      <child link="${prefix}shoulder_link"/>
+      <origin xyz="0.0 0.0 ${shoulder_height}" rpy="0.0 0.0 0.0"/>
+      <axis xyz="0 0 1"/>
       <xacro:unless value="${joint_limited}">
         <limit lower="${-2.0 * pi}" upper="${2.0 * pi}" effort="150.0" velocity="3.15"/>
@@ -112,24 +120,24 @@
       <visual>
         <geometry>
-          <mesh filename="package://ur_description/meshes/ur5/visual/shoulder.dae" />
-        </geometry>
-        <material name="LightGrey">
-          <color rgba="0.7 0.7 0.7 1.0"/>
-        </material>
-      </visual>
-      <collision>
-        <geometry>
-          <mesh filename="package://ur_description/meshes/ur5/collision/shoulder.stl" />
+          <mesh filename="package://ur_description/meshes/ur5/visual/shoulder.dae"/>
+        </geometry>
+        <material name="LightGrey">
+          <color rgba="0.7 0.7 0.7 1.0"/>
+        </material>
+      </visual>
+      <collision>
+        <geometry>
+          <mesh filename="package://ur_description/meshes/ur5/collision/shoulder.stl"/>
         </geometry>
       </collision>
       <xacro:cylinder_inertial radius="0.06" length="0.15" mass="${shoulder_mass}">
-        <origin xyz="0.0 0.0 0.0" rpy="0 0 0" />
+        <origin xyz="0.0 0.0 0.0" rpy="0 0 0"/>
       </xacro:cylinder_inertial>
     </link>
     <joint name="${prefix}shoulder_lift_joint" type="revolute">
-      <parent link="${prefix}shoulder_link" />
-      <child link = "${prefix}upper_arm_link" />
-      <origin xyz="0.0 ${shoulder_offset} 0.0" rpy="0.0 ${pi / 2.0} 0.0" />
-      <axis xyz="0 1 0" />
+      <parent link="${prefix}shoulder_link"/>
+      <child link="${prefix}upper_arm_link"/>
+      <origin xyz="0.0 ${shoulder_offset} 0.0" rpy="0.0 ${pi / 2.0} 0.0"/>
+      <axis xyz="0 1 0"/>
       <xacro:unless value="${joint_limited}">
         <limit lower="${-2.0 * pi}" upper="${2.0 * pi}" effort="150.0" velocity="3.15"/>
@@ -143,24 +151,24 @@
       <visual>
         <geometry>
-          <mesh filename="package://ur_description/meshes/ur5/visual/upperarm.dae" />
-        </geometry>
-        <material name="LightGrey">
-          <color rgba="0.7 0.7 0.7 1.0"/>
-        </material>
-      </visual>
-      <collision>
-        <geometry>
-          <mesh filename="package://ur_description/meshes/ur5/collision/upperarm.stl" />
+          <mesh filename="package://ur_description/meshes/ur5/visual/upperarm.dae"/>
+        </geometry>
+        <material name="LightGrey">
+          <color rgba="0.7 0.7 0.7 1.0"/>
+        </material>
+      </visual>
+      <collision>
+        <geometry>
+          <mesh filename="package://ur_description/meshes/ur5/collision/upperarm.stl"/>
         </geometry>
       </collision>
       <xacro:cylinder_inertial radius="0.06" length="0.56" mass="${upper_arm_mass}">
-        <origin xyz="0.0 0.0 0.28" rpy="0 0 0" />
+        <origin xyz="0.0 0.0 0.28" rpy="0 0 0"/>
       </xacro:cylinder_inertial>
     </link>
     <joint name="${prefix}elbow_joint" type="revolute">
-      <parent link="${prefix}upper_arm_link" />
-      <child link = "${prefix}forearm_link" />
-      <origin xyz="0.0 ${elbow_offset} ${upper_arm_length}" rpy="0.0 0.0 0.0" />
-      <axis xyz="0 1 0" />
+      <parent link="${prefix}upper_arm_link"/>
+      <child link="${prefix}forearm_link"/>
+      <origin xyz="0.0 ${elbow_offset} ${upper_arm_length}" rpy="0.0 0.0 0.0"/>
+      <axis xyz="0 1 0"/>
       <xacro:unless value="${joint_limited}">
         <limit lower="${-pi}" upper="${pi}" effort="150.0" velocity="3.15"/>
@@ -174,24 +182,24 @@
       <visual>
         <geometry>
-          <mesh filename="package://ur_description/meshes/ur5/visual/forearm.dae" />
-        </geometry>
-        <material name="LightGrey">
-          <color rgba="0.7 0.7 0.7 1.0"/>
-        </material>
-      </visual>
-      <collision>
-        <geometry>
-          <mesh filename="package://ur_description/meshes/ur5/collision/forearm.stl" />
+          <mesh filename="package://ur_description/meshes/ur5/visual/forearm.dae"/>
+        </geometry>
+        <material name="LightGrey">
+          <color rgba="0.7 0.7 0.7 1.0"/>
+        </material>
+      </visual>
+      <collision>
+        <geometry>
+          <mesh filename="package://ur_description/meshes/ur5/collision/forearm.stl"/>
         </geometry>
       </collision>
       <xacro:cylinder_inertial radius="0.06" length="0.5" mass="${forearm_mass}">
-        <origin xyz="0.0 0.0 0.25" rpy="0 0 0" />
+        <origin xyz="0.0 0.0 0.25" rpy="0 0 0"/>
       </xacro:cylinder_inertial>
     </link>
     <joint name="${prefix}wrist_1_joint" type="revolute">
-      <parent link="${prefix}forearm_link" />
-      <child link = "${prefix}wrist_1_link" />
-      <origin xyz="0.0 0.0 ${forearm_length}" rpy="0.0 ${pi / 2.0} 0.0" />
-      <axis xyz="0 1 0" />
+      <parent link="${prefix}forearm_link"/>
+      <child link="${prefix}wrist_1_link"/>
+      <origin xyz="0.0 0.0 ${forearm_length}" rpy="0.0 ${pi / 2.0} 0.0"/>
+      <axis xyz="0 1 0"/>
       <xacro:unless value="${joint_limited}">
         <limit lower="${-2.0 * pi}" upper="${2.0 * pi}" effort="28.0" velocity="3.2"/>
@@ -205,24 +213,24 @@
       <visual>
         <geometry>
-          <mesh filename="package://ur_description/meshes/ur5/visual/wrist1.dae" />
-        </geometry>
-        <material name="LightGrey">
-          <color rgba="0.7 0.7 0.7 1.0"/>
-        </material>
-      </visual>
-      <collision>
-        <geometry>
-          <mesh filename="package://ur_description/meshes/ur5/collision/wrist1.stl" />
+          <mesh filename="package://ur_description/meshes/ur5/visual/wrist1.dae"/>
+        </geometry>
+        <material name="LightGrey">
+          <color rgba="0.7 0.7 0.7 1.0"/>
+        </material>
+      </visual>
+      <collision>
+        <geometry>
+          <mesh filename="package://ur_description/meshes/ur5/collision/wrist1.stl"/>
         </geometry>
       </collision>
       <xacro:cylinder_inertial radius="0.6" length="0.12" mass="${wrist_1_mass}">
-        <origin xyz="0.0 0.0 0.0" rpy="0 0 0" />
+        <origin xyz="0.0 0.0 0.0" rpy="0 0 0"/>
       </xacro:cylinder_inertial>
     </link>
     <joint name="${prefix}wrist_2_joint" type="revolute">
-      <parent link="${prefix}wrist_1_link" />
-      <child link = "${prefix}wrist_2_link" />
-      <origin xyz="0.0 ${wrist_1_length} 0.0" rpy="0.0 0.0 0.0" />
-      <axis xyz="0 0 1" />
+      <parent link="${prefix}wrist_1_link"/>
+      <child link="${prefix}wrist_2_link"/>
+      <origin xyz="0.0 ${wrist_1_length} 0.0" rpy="0.0 0.0 0.0"/>
+      <axis xyz="0 0 1"/>
       <xacro:unless value="${joint_limited}">
         <limit lower="${-2.0 * pi}" upper="${2.0 * pi}" effort="28.0" velocity="3.2"/>
@@ -236,24 +244,24 @@
       <visual>
         <geometry>
-          <mesh filename="package://ur_description/meshes/ur5/visual/wrist2.dae" />
-        </geometry>
-        <material name="LightGrey">
-          <color rgba="0.7 0.7 0.7 1.0"/>
-        </material>
-      </visual>
-      <collision>
-        <geometry>
-          <mesh filename="package://ur_description/meshes/ur5/collision/wrist2.stl" />
+          <mesh filename="package://ur_description/meshes/ur5/visual/wrist2.dae"/>
+        </geometry>
+        <material name="LightGrey">
+          <color rgba="0.7 0.7 0.7 1.0"/>
+        </material>
+      </visual>
+      <collision>
+        <geometry>
+          <mesh filename="package://ur_description/meshes/ur5/collision/wrist2.stl"/>
         </geometry>
       </collision>
       <xacro:cylinder_inertial radius="0.6" length="0.12" mass="${wrist_2_mass}">
-        <origin xyz="0.0 0.0 0.0" rpy="0 0 0" />
+        <origin xyz="0.0 0.0 0.0" rpy="0 0 0"/>
       </xacro:cylinder_inertial>
     </link>
     <joint name="${prefix}wrist_3_joint" type="revolute">
-      <parent link="${prefix}wrist_2_link" />
-      <child link = "${prefix}wrist_3_link" />
-      <origin xyz="0.0 0.0 ${wrist_2_length}" rpy="0.0 0.0 0.0" />
-      <axis xyz="0 1 0" />
+      <parent link="${prefix}wrist_2_link"/>
+      <child link="${prefix}wrist_3_link"/>
+      <origin xyz="0.0 0.0 ${wrist_2_length}" rpy="0.0 0.0 0.0"/>
+      <axis xyz="0 1 0"/>
       <xacro:unless value="${joint_limited}">
         <limit lower="${-2.0 * pi}" upper="${2.0 * pi}" effort="28.0" velocity="3.2"/>
@@ -267,23 +275,23 @@
       <visual>
         <geometry>
-          <mesh filename="package://ur_description/meshes/ur5/visual/wrist3.dae" />
-        </geometry>
-        <material name="LightGrey">
-          <color rgba="0.7 0.7 0.7 1.0"/>
-        </material>
-      </visual>
-      <collision>
-        <geometry>
-          <mesh filename="package://ur_description/meshes/ur5/collision/wrist3.stl" />
+          <mesh filename="package://ur_description/meshes/ur5/visual/wrist3.dae"/>
+        </geometry>
+        <material name="LightGrey">
+          <color rgba="0.7 0.7 0.7 1.0"/>
+        </material>
+      </visual>
+      <collision>
+        <geometry>
+          <mesh filename="package://ur_description/meshes/ur5/collision/wrist3.stl"/>
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