Commit message: Restructuration en 3 packages

File: ur_icam_description/urdf/ur5_robotiq85_gripper.urdf.xacro (robot description, xacro)
@@ -1,13 +1,13 @@
 <?xml version="1.0"?>
 <robot name="ur5" xmlns:xacro="http://www.ros.org/wiki/xacro">
-  <xacro:include filename="$(find ur5_description)/urdf/ur5_joint_limited_robot.urdf.xacro" />
-  <xacro:include filename="$(find robotiq_description)/urdf/robotiq_85_gripper.urdf.xacro" />
+  <xacro:include filename="$(find ur_description)/urdf/ur5.urdf.xacro"/>
+  <xacro:include filename="$(find robotiq_description)/urdf/robotiq_85_gripper.urdf.xacro"/>
   <!-- Robotiq Coupler -->
-  <!--  + Height added by the coupler: 8mm -->
-  <!--  + Reference frame: at the middle (4mm) -->
+  <!-- + Height added by the coupler: 8mm -->
+  <!-- + Reference frame: at the middle (4mm) -->
   <link name="robotiq_coupler">
     <visual>
       <geometry>
-        <mesh filename="package://robotiq_description/meshes/robotiq_85_coupler.stl" />
+        <mesh filename="package://robotiq_description/meshes/robotiq_85_coupler.stl"/>
       </geometry>
       <material name="flat_black"/>
@@ -15,16 +15,15 @@
     <collision>
       <geometry>
-        <mesh filename="package://robotiq_description/meshes/robotiq_85_coupler.stl" />
+        <mesh filename="package://robotiq_description/meshes/robotiq_85_coupler.stl"/>
       </geometry>
     </collision>
     <inertial>
-      <origin xyz="2.073e-05   1.45286e-03  -1.1049e-03" rpy="0 0 0" />
-      <mass value="0.168" />
-      <inertia ixx="6.69695624e-05" ixy="5.21511788e-09" ixz="-2.74383009e-08"
-               iyy="7.85088161e-05" iyz="5.41105193e-07" izz="1.41819717e-04"/>
+      <origin xyz="2.073e-05   1.45286e-03  -1.1049e-03" rpy="0 0 0"/>
+      <mass value="0.168"/>
+      <inertia ixx="6.69695624e-05" ixy="5.21511788e-09" ixz="-2.74383009e-08" iyy="7.85088161e-05" iyz="5.41105193e-07" izz="1.41819717e-04"/>
     </inertial>
   </link>
   <joint name="robotiq_coupler_joint" type="fixed">
-    <origin xyz="0 0 0.004" rpy="0 0 ${-pi/2.0}" />
+    <origin xyz="0 0 0.004" rpy="0 0 ${-pi/2.0}"/>
     <parent link="tool0"/>
     <child link="robotiq_coupler"/>
@@ -38,10 +37,10 @@
   <!-- <link name="denso_robotiq_85_gripper" /> -->
   <!-- <joint name="manipulator_dummy_joint" type="fixed"> -->
-  <!--   <origin xyz="0 0 0.1441" rpy="0 0 0" /> -->
-  <!--   <parent link="robotiq_coupler"/> -->
-  <!--   <child link="denso_robotiq_85_gripper"/> -->
+  <!-- <origin xyz="0 0 0.1441" rpy="0 0 0" /> -->
+  <!-- <parent link="robotiq_coupler"/> -->
+  <!-- <child link="denso_robotiq_85_gripper"/> -->
   <!-- </joint> -->
   <!-- Attach the robotiq 85 gripper -->
-  <xacro:robotiq_85_gripper prefix="" parent="robotiq_coupler" >
+  <xacro:robotiq_85_gripper prefix="" parent="robotiq_coupler">
     <origin xyz="0 0 0.004" rpy="0 ${-pi/2} ${pi}"/>
   </xacro:robotiq_85_gripper>
@@ -58,10 +57,12 @@
     </plugin>
   </gazebo>
-  <!-- Gazebo grasping plugin -->
+  <!-- Gazebo grasping plugin
   <gazebo>
     <gripper name="gazebo_gripper">
       <grasp_check>
-        <attach_steps>2</attach_steps>    <!-- default: 20 -->
-        <detach_steps>2</detach_steps>    <!-- default: 40 -->
+        <attach_steps>2</attach_steps>
+        <!- default: 20 ->
+        <detach_steps>2</detach_steps>
+        <!- default: 40 ->
         <min_contact_count>3</min_contact_count>
       </grasp_check>
@@ -71,3 +72,47 @@
     </gripper>
   </gazebo>
+-->
+  <!-- Gazebo grasping plugin  -->
+<gazebo>
+   <plugin name="gazebo_grasp_fix" filename="libgazebo_grasp_fix.so">
+        <arm>
+           <arm_name>ur_arm</arm_name>
+           <palm_link>wrist_3_link</palm_link>
+           <gripper_link>robotiq_85_left_finger_tip_link</gripper_link>
+           <gripper_link>robotiq_85_right_finger_tip_link</gripper_link>
+           <gripper_link>robotiq_85_left_inner_knuckle_link</gripper_link>
+           <gripper_link>robotiq_85_right_inner_knuckle_link</gripper_link>
+           <gripper_link>robotiq_85_left_knuckle_link</gripper_link>
+           <gripper_link>robotiq_85_right_knuckle_link</gripper_link>
+        </arm>
+       <forces_angle_tolerance>100</forces_angle_tolerance>
+       <update_rate>4</update_rate>
+       <grip_count_threshold>4</grip_count_threshold>
+       <max_grip_count>8</max_grip_count>
+       <release_tolerance>0.005</release_tolerance>
+       <disable_collisions_on_attach>false</disable_collisions_on_attach>
+       <contact_topic>__default_topic__</contact_topic>
+    </plugin>
+</gazebo>
+  <!-- Grasping frame -->
+  <link name="grasping_frame">
+    <inertial>
+      <origin xyz="0 0 0" rpy="0 0 0"/>
+      <mass value="0.0001"/>
+      <cuboid_inertia mass="0.0001" x="0.001" y="0.001" z="0.001"/>
+      <inertia ixx="1.0" ixy="0.0" ixz="0.0" iyy="100.0" iyz="0.0" izz="1.0"/>
+    </inertial>
+    <visual>
+      <origin xyz="0 0 0"/>
+      <geometry>
+        <box size="0.01 0.01 0.01"/>
+      </geometry>
+      <material name="White"/>
+    </visual>
+  </link>
+  <joint name="grasping_frame_joint" type="fixed">
+    <parent link="robotiq_coupler"/>
+    <child link="grasping_frame"/>
+    <origin xyz="0 0 0.15" rpy="0 0 0"/>
+  </joint>
 </robot>

Commit message: "update ur_icam package + news ROS drivers"

File: ur_icam_description/urdf/ur5_robotiq85_gripper.urdf.xacro (robot description, xacro)
@@ -86,5 +86,5 @@
            <gripper_link>robotiq_85_right_knuckle_link</gripper_link>
         </arm>
-       <forces_angle_tolerance>100</forces_angle_tolerance>
+       <forces_angle_tolerance>90</forces_angle_tolerance>
        <update_rate>4</update_rate>
        <grip_count_threshold>4</grip_count_threshold>
@@ -105,8 +105,9 @@
     <visual>
       <origin xyz="0 0 0"/>
+      <!-- delete geometry because of collisions between the cube and the gripper when we closed it
       <geometry>
-        <box size="0.01 0.01 0.01"/>
+        <box size="0.001 0.001 0.001"/>
       </geometry>
-      <material name="White"/>
+      <material name="White"/>-->
     </visual>
   </link>
